File: eagle-design/pulse-oximeter.brd (EAGLE design)
At the start: 160 x 100 mm, 9 parts

Commit message: Added new design
Parts:
- moved U$1 72.7 mm to (19.1, 82.5), turned to 90 degrees
- moved JP3 32.5 mm to (39.4, 82.5), turned to 90 degrees
- moved LED4 31.9 mm to (53.3, 68.6), turned to 90 degrees
- moved LED3 28.5 mm to (40.6, 68.6), turned to 90 degrees
- moved R4 23.3 mm to (53.3, 58.4), turned to 90 degrees
- moved R3 14.5 mm to (40.6, 58.4), turned to 90 degrees
- moved JP1 1.27 mm to (49.5, 29.2)
Routing:
- net GND: track 0.00 -> 221.2 mm
- net VCC3.3V: track 0.00 -> 128.9 mm
- net SDA: track 0.00 -> 77.8 mm
- net SCL: track 0.00 -> 74.8 mm, vias 0 -> 1
- net VCC5V: track 0.00 -> 48.2 mm
- net 3V: track 0.00 -> 39.2 mm
- net D5: track 0.00 -> 39.1 mm
- net D4: track 0.00 -> 18.8 mm
- net BATT+: track 0.00 -> 10.2 mm
- net BATT-: track 0.00 -> 8.97 mm
- net N$2: track 0.00 -> 3.01 mm
- net N$1: track 0.00 -> 3.01 mm
Other:
- board size 160 x 100 mm -> 60.9 x 100 mm

Commit message: Updated board design
Parts:
- moved R3 9.14 mm to (40.6, 49.3)
- moved R4 8.89 mm to (53.3, 49.5)
- moved LED3 6.35 mm to (40.6, 62.2)
- moved LED4 6.35 mm to (53.3, 62.2)
Routing:
- net D4: track 18.8 -> 9.63 mm
- net D5: track 39.1 -> 30.2 mm
- net GND: track 221.2 -> 227.6 mm
- net N$1: track 3.01 -> 5.80 mm
- net N$2: track 3.01 -> 5.55 mm
Other:
- outline, holes or cut-outs redrawn
- board text added: "+"
- board text added: "0.98 Inch OLED Display"
- board text added: "220Ω"
- board text added: "3.3V"
- board text added: "BAT +"
- board text added: "BAT -"
- board text added: "Display Error"
- board text added: "GND"
- board text added: "MAX30100 Sensor"
- board text added: "NodeMCU"
- board text added: "Pulse Oximeter"
- board text added: "SCL"
- board text added: "SDA"
- board text added: "Sensor Error"
- board text added: "sashwat.in | github.com/sashuu6"
